File: kicad/velocomp.kicad_pcb (KiCad board)
At the start: 2 copper layers, 45 x 30 mm, 31 parts, among them IC1 STM8S003F3P, J1 USB_B, J2 h2_g, J3 prg, J4 h2, J5 kn1, J6 kn1, Q1 2N7002, SW1 SW_PUSH, SW2 Herkon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

Commit message: start
Parts:
- C2, C4: value 1u -> 1uf
- SP1: footprint Buzzers_Beepers:MagneticBuzzer_ProSignal_ABI-009-RC -> mylibpcb:hc0903a; moved to F.Cu
- moved Q1 3.37 mm to (78.8, 76.3), turned to 180 degrees
- moved SP1 2.18 mm to (77.3, 73.4)
Routing:
- net /spk: track 51.4 -> 48.4 mm
- net VDD: track 47.9 -> 49.6 mm
- net Net-(Q1-Pad3): track 4.48 -> 3.39 mm

Commit message: start
Parts:
- added R4: 10k, Resistors_SMD:R_0603_HandSoldering, B.Cu at (82.4, 68.2)
Routing:
- net GND: track 73.7 -> 76.9 mm
- net /spk: track 48.4 -> 45.4 mm
Changed lines of the file:
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@@
 (kicad_pcb (version 4) (host pcbnew 4.0.7)
   (general
-    (links 67)
-    (no_connects 1)
+    (links 69)
+    (no_connects 2)
     (area 69.924999 49.924999 115.075001 80.075001)
     (thickness 1.6)
     (drawings 5)
-    (tracks 250)
+    (tracks 255)
     (zones 0)
-    (modules 31)
+    (modules 32)
     (nets 34)
   )
@@
     (aux_axis_origin 96.56 130.52)
     (grid_origin 137.16 109.22)
-    (visible_elements 7FFC77FF)
+    (visible_elements 7FFCB7FF)
     (pcbplotparams
       (layerselection 0x00000_80000001)
@@
     )
   )
+  (module Resistors_SMD:R_0603_HandSoldering (layer B.Cu)
+    (at 82.36 68.22 180)
+    (descr "Resistor SMD 0603, hand soldering")
+    (tags "resistor 0603")
+    (attr smd)
+    (fp_text reference R4 (at 0 1.45 180) (layer B.SilkS)
+      (effects (font (size 1 1) (thickness 0.15)) (justify mirror))
+    )
+    (fp_text value 10k (at 0 -1.55 180) (layer B.Fab)
+      (effects (font (size 1 1) (thickness 0.15)) (justify mirror))
+    )
+    (fp_text user %R (at 0 0 180) (layer B.Fab)
+      (effects (font (size 0.4 0.4) (thickness 0.075)) (justify mirror))
+    )
+    (fp_line (start -0.8 -0.4) (end -0.8 0.4) (layer B.Fab) (width 0.1))
+    (fp_line (start 0.8 -0.4) (end -0.8 -0.4) (layer B.Fab) (width 0.1))
+    (fp_line (start 0.8 0.4) (end 0.8 -0.4) (layer B.Fab) (width 0.1))
+    (fp_line (start -0.8 0.4) (end 0.8 0.4) (layer B.Fab) (width 0.1))
+    (fp_line (start 0.5 -0.68) (end -0.5 -0.68) (layer B.SilkS) (width 0.12))
+    (fp_line (start -0.5 0.68) (end 0.5 0.68) (layer B.SilkS) (width 0.12))
+    (fp_line (start -1.96 0.7) (end 1.95 0.7) (layer B.CrtYd) (width 0.05))
+    (fp_line (start -1.96 0.7) (end -1.96 -0.7) (layer B.CrtYd) (width 0.05))
+    (fp_line (start 1.95 -0.7) (end 1.95 0.7) (layer B.CrtYd) (width 0.05))
+    (fp_line (start 1.95 -0.7) (end -1.96 -0.7) (layer B.CrtYd) (width 0.05))
+    (pad 1 smd rect (at -1.1 0 180) (size 1.2 0.9) (layers B.Cu B.Paste B.Mask)
+      (net 27 /spk))
+    (pad 2 smd rect (at 1.1 0 180) (size 1.2 0.9) (layers B.Cu B.Paste B.Mask)
+      (net 1 GND))
+    (model ${KISYS3DMOD}/Resistors_SMD.3dshapes/R_0603.wrl
+      (at (xyz 0 0 0))
+      (scale (xyz 1 1 1))
+      (rotate (xyz 0 0 0))
+    )
+  )
   (gr_circle (center 95.52 62.84) (end 95.52 74.84) (layer F.SilkS) (width 0.2))
   (gr_line (start 114.16 50) (end 114.16 80) (angle 90) (layer Edge.Cuts) (width 0.15))
@@
   (gr_line (start 70 50) (end 70 80) (angle 90) (layer Edge.Cuts) (width 0.15))
   (gr_line (start 70 50) (end 115 50) (angle 90) (layer Edge.Cuts) (width 0.15))
+  (segment (start 87.36 74.32) (end 89.26 74.32) (width 0.3) (layer F.Cu) (net 1))
+  (segment (start 89.51 74.07) (end 89.51 73.12) (width 0.3) (layer F.Cu) (net 1))
+  (segment (start 89.26 74.32) (end 89.51 74.07) (width 0.3) (layer F.Cu) (net 1))
   (segment (start 73.96 65.52) (end 73.96 59.42) (width 0.3) (layer F.Cu) (net 1))
   (segment (start 111.26 52.92) (end 111.26 52.5) (width 0.2) (layer B.Cu) (net 1))
@@
   (via (at 88.66 76.52) (size 2) (drill 0.8) (layers F.Cu B.Cu) (net 24))
   (segment (start 88.66 76.52) (end 88.56 76.52) (width 0.2) (layer F.Cu) (net 24))
+  (segment (start 85.16 76.52) (end 85.16 73.42) (width 0.3) (layer B.Cu) (net 27))
+  (segment (start 83.46 59.22) (end 84.46 58.22) (width 0.3) (layer B.Cu) (net 27))
+  (segment (start 83.46 71.72) (end 83.46 59.22) (width 0.3) (layer B.Cu) (net 27))
+  (segment (start 85.16 73.42) (end 83.46 71.72) (width 0.3) (layer B.Cu) (net 27))
+  (segment (start 85.16 76.52) (end 85.16 74.62) (width 0.3) (layer F.Cu) (net 27))
+  (segment (start 85.16 74.62) (end 84.86 74.32) (width 0.3) (layer F.Cu) (net 27))
   (segment (start 79.76 77.27) (end 81.71 77.27) (width 0.3) (layer F.Cu) (net 27))
   (segment (start 81.71 77.27) (end 82.544375 76.435625) (width 0.3) (layer F.Cu) (net 27))
-  (segment (start 85.16 76.52) (end 81.86 76.42) (width 0.3) (layer B.Cu) (net 27))
-  (segment (start 83.96 58.22) (end 86.36 58.22) (width 0.3) (layer B.Cu) (net 27))
-  (segment (start 79.56 62.62) (end 83.96 58.22) (width 0.3) (layer B.Cu) (net 27))
-  (segment (start 79.56 74.12) (end 79.56 62.62) (width 0.3) (layer B.Cu) (net 27))
-  (segment (start 81.86 76.42) (end 79.56 74.12) (width 0.3) (layer B.Cu) (net 27))
+  (segment (start 84.46 58.22) (end 86.36 58.22) (width 0.3) (layer B.Cu) (net 27))
   (segment (start 86.36 58.22) (end 86.36 58.32) (width 0.3) (layer F.Cu) (net 27))
   (via (at 86.36 58.22) (size 2) (drill 0.8) (layers F.Cu B.Cu) (net 27))

Commit message: start
Parts:
- added J7: ind, mylibpcb:wirepad_mini, F.Cu at (88.9, 62.9)
- added J8: ind, mylibpcb:wirepad_mini, F.Cu at (100.7, 67.4)
- moved J3 1.82 mm to (98.8, 67.4)
Routing:
- net Net-(IC1-Pad19): track 0.00 -> 7.52 mm
- net Net-(IC1-Pad11): track 0.00 -> 2.07 mm
- net /spk: track 45.4 -> 43.6 mm
- net Net-(Q1-Pad3): track 3.39 -> 4.10 mm

Commit message: start
Parts:
- R2: value 300 -> 1k
- R3: value 1k -> 3k
Connections:
- U2 pad 1: Net-(U2-Pad1) -> GND
Routing:
- net GND: track 76.9 -> 80.2 mm

Commit message: start
Parts:
- removed R3: 3k, Resistors_SMD:R_0603_HandSoldering
Connections:
- D2 pad 4: Net-(D2-Pad4) -> (no net)
- IC1 pad 12: Net-(IC1-Pad12) -> (no net)
- IC1 pad 14: Net-(IC1-Pad14) -> (no net)
- IC1 pad 15: Net-(IC1-Pad15) -> (no net)
- IC1 pad 4: Net-(IC1-Pad4) -> (no net)
- J1 pad 2: Net-(J1-Pad2) -> (no net)
- J1 pad 3: Net-(J1-Pad3) -> (no net)
- U1 pad 11: Net-(U1-Pad11) -> (no net)
- U2 pad 6: Net-(U2-Pad6) -> (no net)
Routing:
- net Net-(IC1-Pad4): track 5.94 -> 0.00 mm
- net (no net): track 0.00 -> 5.94 mm
