File: kicad/velocomp.sch (KiCad schematic (older format))
At the start: 29 parts, among them IC1 STM8S003F3P, J1 USB_B, J2 h2_g, J3 prg, J4 h2, J5 kn1, J6 kn1, Q1 2N7002, SW1 SW_PUSH, SW2 Herkon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

Commit message: start
Parts:
- SP1: footprint Buzzers_Beepers:MagneticBuzzer_ProSignal_ABI-009-RC -> mylibpcb:hc0903a
Changed lines of the file:
@@
 F 0 "SP1" H 7300 1350 50  0000 C CNN
 F 1 "HC0903A" H 7300 850 50  0000 C CNN
-F 2 "Buzzers_Beepers:MagneticBuzzer_ProSignal_ABI-009-RC" H 7400 1100 50  0000 C CNN
+F 2 "mylibpcb:hc0903a" H 7400 1100 50  0000 C CNN
 F 3 "" H 7400 1100 50  0000 C CNN
 	1    7400 1100

Commit message: start
Parts:
- added R4: 10k, Resistors_SMD:R_0603_HandSoldering, symbol R_Small
Connections:
- net GND: now also R4.2
- net spk: now also R4.1
Changed lines of the file:
@@
 $EndComp
 $Comp
-L GND #PWR01
+L GND #PWR7
 U 1 1 5778E13F
 P 3550 1400
-F 0 "#PWR01" H 3550 1150 50  0001 C CNN
+F 0 "#PWR7" H 3550 1150 50  0001 C CNN
 F 1 "GND" H 3550 1250 50  0000 C CNN
 F 2 "" H 3550 1400 50  0000 C CNN
@@
 $EndComp
 $Comp
-L VDD #PWR02
+L VDD #PWR5
 U 1 1 5778E176
 P 3450 1200
-F 0 "#PWR02" H 3450 1050 50  0001 C CNN
+F 0 "#PWR5" H 3450 1050 50  0001 C CNN
 F 1 "VDD" H 3450 1350 50  0000 C CNN
 F 2 "" H 3450 1200 50  0000 C CNN
@@
 H2
 $Comp
-L GND #PWR03
+L GND #PWR10
 U 1 1 577CA99E
 P 4350 4550
-F 0 "#PWR03" H 4350 4300 50  0001 C CNN
+F 0 "#PWR10" H 4350 4300 50  0001 C CNN
 F 1 "GND" H 4350 4400 50  0000 C CNN
 F 2 "" H 4350 4550 50  0000 C CNN
@@
 $EndComp
 $Comp
-L GND #PWR04
+L GND #PWR12
 U 1 1 577CB28E
 P 5050 4700
-F 0 "#PWR04" H 5050 4450 50  0001 C CNN
+F 0 "#PWR12" H 5050 4450 50  0001 C CNN
 F 1 "GND" H 5050 4550 50  0000 C CNN
 F 2 "" H 5050 4700 50  0000 C CNN
@@
 $EndComp
 $Comp
-L GND #PWR05
+L GND #PWR15
 U 1 1 577CB3DD
 P 6250 4500
-F 0 "#PWR05" H 6250 4250 50  0001 C CNN
+F 0 "#PWR15" H 6250 4250 50  0001 C CNN
 F 1 "GND" H 6250 4350 50  0000 C CNN
 F 2 "" H 6250 4500 50  0000 C CNN
@@
 $EndComp
 $Comp
-L VDD #PWR06
+L VDD #PWR14
 U 1 1 577CB448
 P 5900 3700
-F 0 "#PWR06" H 5900 3550 50  0001 C CNN
+F 0 "#PWR14" H 5900 3550 50  0001 C CNN
 F 1 "VDD" H 5900 3850 50  0000 C CNN
 F 2 "" H 5900 3700 50  0000 C CNN
@@
 RX
 $Comp
-L GND #PWR07
+L GND #PWR11
 U 1 1 577D2AAC
 P 4350 6600
-F 0 "#PWR07" H 4350 6350 50  0001 C CNN
+F 0 "#PWR11" H 4350 6350 50  0001 C CNN
 F 1 "GND" H 4350 6450 50  0000 C CNN
 F 2 "" H 4350 6600 50  0000 C CNN
@@
 $EndComp
 $Comp
-L GND #PWR08
+L GND #PWR6
 U 1 1 57907976
 P 3500 3350
-F 0 "#PWR08" H 3500 3100 50  0001 C CNN
+F 0 "#PWR6" H 3500 3100 50  0001 C CNN
 F 1 "GND" H 3500 3200 50  0000 C CNN
 F 2 "" H 3500 3350 50  0000 C CNN
@@
 $EndComp
 $Comp
-L GND #PWR09
+L GND #PWR4
 U 1 1 57AD96D3
 P 2100 3250
-F 0 "#PWR09" H 2100 3000 50  0001 C CNN
+F 0 "#PWR4" H 2100 3000 50  0001 C CNN
 F 1 "GND" H 2100 3100 50  0000 C CNN
 F 2 "" H 2100 3250 50  0000 C CNN
@@
 5v
 $Comp
-L GND #PWR010
+L GND #PWR1
 U 1 1 57AD9E56
 P 1400 4500
-F 0 "#PWR010" H 1400 4250 50  0001 C CNN
+F 0 "#PWR1" H 1400 4250 50  0001 C CNN
 F 1 "GND" H 1400 4350 50  0000 C CNN
 F 2 "" H 1400 4500 50  0000 C CNN
@@
 $EndComp
 $Comp
-L GND #PWR011
+L GND #PWR2
 U 1 1 57ADA085
 P 1550 4950
-F 0 "#PWR011" H 1550 4700 50  0001 C CNN
+F 0 "#PWR2" H 1550 4700 50  0001 C CNN
 F 1 "GND" H 1550 4800 50  0000 C CNN
 F 2 "" H 1550 4950 50  0000 C CNN
@@
 $EndComp
 $Comp
-L GND #PWR012
+L GND #PWR13
 U 1 1 57ADDF9F
 P 5550 1500
-F 0 "#PWR012" H 5550 1250 50  0001 C CNN
+F 0 "#PWR13" H 5550 1250 50  0001 C CNN
 F 1 "GND" H 5550 1350 50  0000 C CNN
 F 2 "" H 5550 1500 50  0000 C CNN
@@
 Connection ~ 5100 1950
 $Comp
-L GND #PWR013
+L GND #PWR16
 U 1 1 57ADEF4C
 P 6900 2750
-F 0 "#PWR013" H 6900 2500 50  0001 C CNN
+F 0 "#PWR16" H 6900 2500 50  0001 C CNN
 F 1 "GND" H 6900 2600 50  0000 C CNN
 F 2 "" H 6900 2750 50  0000 C CNN
@@
 	3800 4250 5050 4250
 $Comp
-L VDD #PWR014
+L VDD #PWR9
 U 1 1 5974CA85
 P 4350 4100
-F 0 "#PWR014" H 4350 3950 50  0001 C CNN
+F 0 "#PWR9" H 4350 3950 50  0001 C CNN
 F 1 "VDD" H 4350 4250 50  0000 C CNN
 F 2 "" H 4350 4100 50  0001 C CNN
@@
 5v
 $Comp
-L GND #PWR015
+L GND #PWR3
 U 1 1 5974DCC0
 P 1600 6750
-F 0 "#PWR015" H 1600 6500 50  0001 C CNN
+F 0 "#PWR3" H 1600 6500 50  0001 C CNN
 F 1 "GND" H 1600 6600 50  0000 C CNN
 F 2 "" H 1600 6750 50  0001 C CNN
@@
 H1
 $Comp
-L GND #PWR016
+L GND #PWR20
 U 1 1 5974E707
 P 8850 3450
-F 0 "#PWR016" H 8850 3200 50  0001 C CNN
+F 0 "#PWR20" H 8850 3200 50  0001 C CNN
 F 1 "GND" H 8850 3300 50  0000 C CNN
 F 2 "" H 8850 3450 50  0001 C CNN
@@
 $EndComp
 $Comp
-L GND #PWR017
+L GND #PWR19
 U 1 1 5974ED9E
 P 8450 3750
-F 0 "#PWR017" H 8450 3500 50  0001 C CNN
+F 0 "#PWR19" H 8450 3500 50  0001 C CNN
 F 1 "GND" H 8450 3600 50  0000 C CNN
 F 2 "" H 8450 3750 50  0000 C CNN
@@
 $EndComp
 $Comp
-L GND #PWR018
+L GND #PWR18
 U 1 1 599A8CA0
 P 7700 2050
-F 0 "#PWR018" H 7700 1800 50  0001 C CNN
+F 0 "#PWR18" H 7700 1800 50  0001 C CNN
 F 1 "GND" H 7700 1900 50  0000 C CNN
 F 2 "" H 7700 2050 50  0001 C CNN
@@
 spk
 $Comp
-L VDD #PWR019
+L VDD #PWR17
 U 1 1 599A8E61
 P 7700 1000
-F 0 "#PWR019" H 7700 850 50  0001 C CNN
+F 0 "#PWR17" H 7700 850 50  0001 C CNN
 F 1 "VDD" H 7700 1150 50  0000 C CNN
 F 2 "" H 7700 1000 50  0001 C CNN
@@
 Connection ~ 3650 5550
 $Comp
-L GND #PWR020
+L GND #PWR8
 U 1 1 59CFE8F1
 P 3650 5950
-F 0 "#PWR020" H 3650 5700 50  0001 C CNN
+F 0 "#PWR8" H 3650 5700 50  0001 C CNN
 F 1 "GND" H 3650 5800 50  0000 C CNN
 F 2 "" H 3650 5950 50  0001 C CNN
@@
 Wire Wire Line
 	4800 2650 5000 2650
+$Comp
+L R_Small R4
+U 1 1 59ECD965
+P 7450 1900
+F 0 "R4" H 7480 1920 50  0000 L CNN
+F 1 "10k" H 7480 1860 50  0000 L CNN
+F 2 "Resistors_SMD:R_0603_HandSoldering" H 7450 1900 50  0001 C CNN
+F 3 "" H 7450 1900 50  0001 C CNN
+	1    7450 1900
+	1    0    0    -1
+$EndComp
+Wire Wire Line
+	7450 2000 7700 2000
+Connection ~ 7700 2000
+Wire Wire Line
+	7450 1800 7450 1700
+Wire Wire Line
+	7450 1700 7400 1700
 $EndSCHEMATC

Commit message: start
Parts:
- added J7, J8: ind, mylibpcb:wirepad_mini, symbol CONN_01X01
Connections:
- net at IC1.11 ([TIM1_BKIN]I2C_SDA/PB5): now also J7.1 (P1)
- net at IC1.19 (PD2/AIN3[TIM2_CH3]): now also J8.1 (P1)
Changed lines of the file:
@@
 Wire Wire Line
 	7450 1700 7400 1700
+$Comp
+L CONN_01X01 J7
+U 1 1 59F37556
+P 5050 2450
+F 0 "J7" H 5050 2550 50  0000 C CNN
+F 1 "ind" V 5150 2450 50  0000 C CNN
+F 2 "mylibpcb:wirepad_mini" H 5050 2450 50  0001 C CNN
+F 3 "" H 5050 2450 50  0001 C CNN
+	1    5050 2450
+	1    0    0    -1
+$EndComp
+Wire Wire Line
+	4800 2450 4850 2450
+$Comp
+L CONN_01X01 J8
+U 1 1 59F37AC9
+P 1950 2350
+F 0 "J8" H 1950 2450 50  0000 C CNN
+F 1 "ind" V 2050 2350 50  0000 C CNN
+F 2 "mylibpcb:wirepad_mini" H 1950 2350 50  0001 C CNN
+F 3 "" H 1950 2350 50  0001 C CNN
+	1    1950 2350
+	-1   0    0    1
+$EndComp
+Wire Wire Line
+	2200 2350 2150 2350
 $EndSCHEMATC

Commit message: start
Parts:
- J1: footprint mylibpcb:usb5s -> myowndevice:usb5s
- R2: value 300 -> 1k
- R3: value 1k -> 3k
- SP1: footprint mylibpcb:hc0903a -> myowndevice:hc0903a
- U1: footprint mylibpcb:hc-05 -> myowndevice:hc-05
Changed lines of the file:
@@
 F 0 "U1" H 4300 5200 60  0000 C CNN
 F 1 "BK3231" H 4700 5200 60  0000 C CNN
-F 2 "mylibpcb:hc-05" H 4500 5200 60  0000 C CNN
+F 2 "myowndevice:hc-05" H 4500 5200 60  0000 C CNN
 F 3 "" H 4500 5200 60  0000 C CNN
 	1    4500 5200
@@
 F 0 "SP1" H 7300 1350 50  0000 C CNN
 F 1 "HC0903A" H 7300 850 50  0000 C CNN
-F 2 "mylibpcb:hc0903a" H 7400 1100 50  0000 C CNN
+F 2 "myowndevice:hc0903a" H 7400 1100 50  0000 C CNN
 F 3 "" H 7400 1100 50  0000 C CNN
 	1    7400 1100
@@
 F 0 "J1" H 1400 6800 50  0000 L CNN
 F 1 "USB_B" H 1400 6700 50  0000 L CNN
-F 2 "mylibpcb:usb5s" H 1750 6300 50  0001 C CNN
+F 2 "myowndevice:usb5s" H 1750 6300 50  0001 C CNN
 F 3 "" H 1750 6300 50  0001 C CNN
 	1    1600 6350
@@
 P 3500 5550
 F 0 "R2" H 3530 5570 50  0000 L CNN
-F 1 "300" H 3530 5510 50  0000 L CNN
+F 1 "1k" H 3530 5510 50  0000 L CNN
 F 2 "Resistors_SMD:R_0603_HandSoldering" H 3500 5550 50  0001 C CNN
 F 3 "" H 3500 5550 50  0001 C CNN
@@
 P 3650 5750
 F 0 "R3" H 3680 5770 50  0000 L CNN
-F 1 "1k" H 3680 5710 50  0000 L CNN
+F 1 "3k" H 3680 5710 50  0000 L CNN
 F 2 "Resistors_SMD:R_0603_HandSoldering" H 3650 5750 50  0001 C CNN
 F 3 "" H 3650 5750 50  0001 C CNN

Commit message: start
Connections:
- net GND: now also U2.1 (TEMP)
- no-connect marks 4 -> 3
Changed lines of the file:
@@
 	0    1    1    0
 $EndComp
-NoConn ~ 1900 4250
 $Comp
 L C_Small C3
@@
 Wire Wire Line
 	2200 2350 2150 2350
+$Comp
+L GND #PWR?
+U 1 1 5A57BC6E
+P 1900 4250
+F 0 "#PWR?" H 1900 4000 50  0001 C CNN
+F 1 "GND" H 1900 4100 50  0000 C CNN
+F 2 "" H 1900 4250 50  0000 C CNN
+F 3 "" H 1900 4250 50  0000 C CNN
+	1    1900 4250
+	0    1    1    0
+$EndComp
 $EndSCHEMATC

Commit message: start
Parts:
- removed R3: 3k, Resistors_SMD:R_0603_HandSoldering, symbol R_Small
- BT1: symbol Battery-RESCUE-velocomp -> velocomp-rescue:Battery-RESCUE-velocomp
- C1, C2, C3, C4, C5, C6, C7, C8: symbol C_Small -> velocomp-rescue:C_Small
- D1: symbol LED_Small -> velocomp-rescue:LED_Small
- D2: symbol NCP603-RESCUE-velocomp -> velocomp-rescue:NCP603-RESCUE-velocomp
- IC1: symbol STM8S003F3P -> velocomp-rescue:STM8S003F3P
- J1: symbol USB_B -> velocomp-rescue:USB_B
- J2, J3, J4, J5, J6, J7, J8: symbol CONN_01X01 -> velocomp-rescue:CONN_01X01
- Q1: symbol Q_NMOS_GSD -> velocomp-rescue:Q_NMOS_GSD
- R1, R4, R6: symbol R_Small -> velocomp-rescue:R_Small
- R2: value 1k -> 10k; symbol R_Small -> velocomp-rescue:R_Small
- SP1: symbol SPEAKER -> velocomp-rescue:SPEAKER
- SW1, SW2: symbol SW_PUSH -> velocomp-rescue:SW_PUSH
- U1: symbol HC-05 -> mylibkicad:HC-05
- U2: symbol TP4056 -> mylibkicad:TP4056
- Y1: symbol Crystal_Small -> velocomp-rescue:Crystal_Small
Other:
- note removed: "Уточнить.! вроде модуль может работать до 4.2в - нам этого и надо! тогда просто транзистор ставим и все!"
- note removed: "выключатель между выв 3мм и между крайними тоже\nвысота 5мм"
- moved on the sheet: J2, J3, J4, J5, J6, R2, SW2, U1
